File: diy-audio/pcb_eagle/OSSC_HDMI_Audio_v1.5_A4b.sch (EAGLE design)
At the start: 29 parts, among them U1 PCM1808, U2 74LVC1G34, U3 MK2507SLF

Commit message: PCB files with a pad for mclk to IT6613E
Parts:
- removed U$4: OSSC_OVERLAY_2, OSSC_HDMI_Audio:OSSC_OVERLAY_2
- added U$1: OSSC_DIY_AUDIO_OVERLAYDIY-V1.5B, OSSC_HDMI_Audio:OSSC_DIY_AUDIO_OVERLAYDIY-V1.5B
Connections:
- net GND: now also U$1G$2.GND; no longer U$4G$2.GND
- net N$1: now also U$1G$2.A_L; no longer U$4G$2.A_L
- net N$13: now also U$1G$1.WS; no longer U$4G$1.WS
- net N$14: now also U$1G$1.SCK; no longer U$4G$1.SCK
- net N$15: now also U$1G$1.I2S0; no longer U$4G$1.I2S0
- net N$17: now also U$1G$1.MCLK
- net N$2: now also U$1G$2.A_R; no longer U$4G$2.A_R
Changed lines of the file:
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@@
 <?xml version="1.0" encoding="utf-8"?>
 <!DOCTYPE eagle SYSTEM "eagle.dtd">
-<eagle version="7.5.0">
+<eagle version="7.6.0">
 <drawing>
 <settings>
@@
 <part name="FB2" library="rcl" deviceset="R-EU_" device="R0603"/>
 <part name="U2" library="OSSC_HDMI_Audio" deviceset="74LVC1G34" device=""/>
-<part name="U$4" library="OSSC_HDMI_Audio" deviceset="OSSC_OVERLAY_2" device=""/>
+<part name="U$1" library="OSSC_HDMI_Audio" deviceset="OSSC_DIY_AUDIO_OVERLAY" device="DIY-V1.5B" value="OSSC_DIY_AUDIO_OVERLAYDIY-V1.5B"/>
 </parts>
 <sheets>
@@
 <instance part="U2" gate="G$1" x="22.86" y="30.48"/>
 <instance part="U2" gate="G$2" x="83.82" y="48.26"/>
-<instance part="U$4" gate="G$1" x="205.74" y="22.86"/>
-<instance part="U$4" gate="G$2" x="208.28" y="60.96"/>
+<instance part="U$1" gate="G$1" x="205.74" y="27.94"/>
+<instance part="U$1" gate="G$2" x="208.28" y="60.96"/>
 </instances>
 <busses>
@@
 <pinref part="GND1" gate="1" pin="GND"/>
 <wire x1="198.12" y1="55.88" x2="198.12" y2="53.34" width="0.1524" layer="91"/>
-<wire x1="200.66" y1="55.88" x2="198.12" y2="55.88" width="0.1524" layer="91"/>
-<pinref part="U$4" gate="G$2" pin="GND"/>
+<pinref part="U$1" gate="G$2" pin="GND"/>
+<wire x1="198.12" y1="55.88" x2="200.66" y2="55.88" width="0.1524" layer="91"/>
 </segment>
 <segment>
@@
 <segment>
 <pinref part="C18" gate="G$1" pin="-"/>
+<pinref part="U$1" gate="G$2" pin="A_L"/>
 <wire x1="200.66" y1="60.96" x2="193.04" y2="60.96" width="0.1524" layer="91"/>
-<pinref part="U$4" gate="G$2" pin="A_L"/>
 </segment>
 </net>
@@
 <segment>
 <pinref part="C17" gate="G$1" pin="-"/>
+<pinref part="U$1" gate="G$2" pin="A_R"/>
 <wire x1="200.66" y1="66.04" x2="193.04" y2="66.04" width="0.1524" layer="91"/>
-<pinref part="U$4" gate="G$2" pin="A_R"/>
 </segment>
 </net>
@@
 <wire x1="134.62" y1="35.56" x2="132.08" y2="35.56" width="0.1524" layer="91"/>
 <wire x1="132.08" y1="35.56" x2="132.08" y2="30.48" width="0.1524" layer="91"/>
-<wire x1="132.08" y1="30.48" x2="200.66" y2="30.48" width="0.1524" layer="91"/>
-<pinref part="U$4" gate="G$1" pin="WS"/>
+<wire x1="132.08" y1="30.48" x2="198.12" y2="30.48" width="0.1524" layer="91"/>
+<pinref part="U$1" gate="G$1" pin="WS"/>
 </segment>
 </net>
 <net name="N$14" class="0">
 <segment>
-<wire x1="162.56" y1="35.56" x2="200.66" y2="35.56" width="0.1524" layer="91"/>
+<wire x1="162.56" y1="35.56" x2="198.12" y2="35.56" width="0.1524" layer="91"/>
 <pinref part="U1" gate="G$1" pin="BCK"/>
-<pinref part="U$4" gate="G$1" pin="SCK"/>
+<pinref part="U$1" gate="G$1" pin="SCK"/>
 </segment>
 </net>
@@
 <wire x1="162.56" y1="40.64" x2="177.8" y2="40.64" width="0.1524" layer="91"/>
 <wire x1="177.8" y1="40.64" x2="177.8" y2="25.4" width="0.1524" layer="91"/>
-<wire x1="177.8" y1="25.4" x2="200.66" y2="25.4" width="0.1524" layer="91"/>
-<pinref part="U$4" gate="G$1" pin="I2S0"/>
+<wire x1="177.8" y1="25.4" x2="198.12" y2="25.4" width="0.1524" layer="91"/>
+<pinref part="U$1" gate="G$1" pin="I2S0"/>
 </segment>
 </net>
@@
 <pinref part="R31" gate="G$1" pin="2"/>
 <wire x1="129.54" y1="30.48" x2="91.44" y2="30.48" width="0.1524" layer="91"/>
-</segment>
-</net>
+<pinref part="U$1" gate="G$1" pin="MCLK"/>
+<wire x1="198.12" y1="20.32" x2="129.54" y2="20.32" width="0.1524" layer="91"/>
+<wire x1="129.54" y1="20.32" x2="129.54" y2="30.48" width="0.1524" layer="91"/>
+<junction x="129.54" y="30.48"/>
+</segment>
+</net>
